File: Roboballers Pcb.kicad_pcb (KiCad board)
At the start: 4 copper layers, 120 x 120 mm, 116 parts, among them J1 Conn_01x02, J2 Conn_01x02, J3 Conn_01x02, J4 Conn_01x02, J5 Screw_Terminal_01x02, J6 Conn_01x02, J7 Bottom_Pcb, SW1 OS102011MS2QN1, SW2 OS102011MS2QN1, SW3 OS102011MS2QN1, SW4 OS102011MS2QN1, U1 VNH7070ASTR, U10 TSOP25xx, U11 OpenMV_H7_R2, U12 MCP3008, U13 TSOP25xx, U14 TSOP25xx, U15 SEN0140, U16 TSOP25xx, U17 RockerSwitch, U18 TSOP25xx, U19 TSOP25xx, U2 VNH7070ASTR, U20 TSOP25xx, U21 TSOP25xx, U22 TSOP25xx, U23 TSOP25xx, U24 TSOP25xx, U25 TSOP25xx, U26 TSOP25xx, U27 MCP3008, U28 MCP3008, U29 TSOP25xx, U3 VNH7070ASTR, U30 TSOP25xx, U31 TSOP25xx, U32 TSOP25xx, U33 TSOP25xx, U34 TSOP25xx, U35 TSOP25xx, U36 TSOP25xx, U4 VNH7070ASTR, U5 Teensy4.1, U6 TSOP25xx, U7 V_Regulator_-_5v, U8 TSOP25xx, U9 TSOP25xx

Commit message: idk
Connections:
- U5 pad 25: unconnected-(U5-33_MCLK2-Pad25) -> CLS1
- U5 pad 26: unconnected-(U5-34_RX8-Pad26) -> CLS2
- U5 pad 27: unconnected-(U5-35_TX8-Pad27) -> CLS3
Routing:
- net CLS2: track 0.00 -> 47.6 mm, vias 0 -> 2
- net CLS3: track 0.00 -> 22.7 mm, vias 0 -> 2
- net CLS1: track 0.00 -> 15.3 mm, vias 0 -> 1
